File: LX3000DMod/Demux.kicad_sch (KiCad schematic)
At the start: 18 parts

Commit message: updated repo and bkp state
Parts:
- C15, C16: renamed from C?; Spice_Model 0.1u -> (none); Spice_Netlist_Enabled Y -> (none); Spice_Primitive C -> (none)
- gave numbers to parts that had none: 16
