File: LX3000DMod/OpAmp.kicad_sch (KiCad schematic)
At the start: 23 parts

Commit message: audio input terminado
Changed lines of the file:
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@@
     (effects (font (size 1.27 1.27)) (justify right))
   )
-  (hierarchical_label "OutA" (shape input) (at 163.83 143.51 0)
+  (hierarchical_label "OutA" (shape output) (at 163.83 143.51 0)
     (effects (font (size 1.27 1.27)) (justify left))
   )
@@
     (effects (font (size 1.27 1.27)) (justify right))
   )
-  (hierarchical_label "OutB" (shape input) (at 162.56 91.44 0)
+  (hierarchical_label "OutB" (shape output) (at 162.56 91.44 0)
     (effects (font (size 1.27 1.27)) (justify left))
   )

Commit message: updated repo and bkp state
Parts:
- C1, C2, C7, C8: renamed from C?; Spice_Model 4.7u -> (none); Spice_Netlist_Enabled Y -> (none); Spice_Primitive C -> (none)
- C4: renamed from C?; Spice_Model 0.1u -> (none); Spice_Netlist_Enabled Y -> (none); Spice_Primitive C -> (none)
- C5, C6: renamed from C?; Spice_Model 47p -> (none); Spice_Netlist_Enabled Y -> (none); Spice_Primitive C -> (none)
- R1, R2, R5, R6: renamed from R?; Spice_Model 100k -> (none); Spice_Netlist_Enabled Y -> (none); Spice_Primitive R -> (none)
- R10, R9: renamed from R?; Spice_Model 12k -> (none); Spice_Netlist_Enabled Y -> (none); Spice_Primitive R -> (none)
- R11, R12: renamed from R?; Spice_Model 4.7k -> (none); Spice_Netlist_Enabled Y -> (none); Spice_Primitive R -> (none)
- R3, R4: renamed from R?; Spice_Model 10k -> (none); Spice_Netlist_Enabled Y -> (none); Spice_Primitive R -> (none)
- R7, R8: renamed from R?; Spice_Model 1k -> (none); Spice_Netlist_Enabled Y -> (none); Spice_Primitive R -> (none)
- gave numbers to parts that had none: 2
