File: UpgradeBoard/OpAmpPsu.kicad_sch (KiCad schematic)
At the start: 6 parts

Commit message: psucorrection
Parts:
- gave numbers to parts that had none: 6
Changed lines of the file:
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@@
   (symbol (lib_id "Device:C") (at 99.06 134.62 0) (unit 1)
     (in_bom yes) (on_board yes) (dnp no) (fields_autoplaced)
-    (property "Reference" "C?" (at 102.87 133.3499 0)
+    (property "Reference" "C19" (at 102.87 133.3499 0)
       (effects (font (size 1.27 1.27)) (justify left))
     )
@@
       (project "UpgradeBoard"
         (path "/32326095-4589-49eb-bfdc-5004b37213a0/3e08591f-9f75-4f14-b240-40be088c15b2"
-          (reference "C?") (unit 1)
+          (reference "C19") (unit 1)
         )
       )
@@
   (symbol (lib_id "Device:R") (at 92.71 130.81 90) (unit 1)
     (in_bom yes) (on_board yes) (dnp no) (fields_autoplaced)
-    (property "Reference" "R?" (at 92.71 124.46 90)
+    (property "Reference" "R20" (at 92.71 124.46 90)
       (effects (font (size 1.27 1.27)))
     )
@@
       (project "UpgradeBoard"
         (path "/32326095-4589-49eb-bfdc-5004b37213a0/3e08591f-9f75-4f14-b240-40be088c15b2"
-          (reference "R?") (unit 1)
+          (reference "R20") (unit 1)
         )
       )
@@
   (symbol (lib_id "Device:C") (at 99.06 152.4 0) (unit 1)
     (in_bom yes) (on_board yes) (dnp no) (fields_autoplaced)
-    (property "Reference" "C?" (at 102.87 151.1299 0)
+    (property "Reference" "C20" (at 102.87 151.1299 0)
       (effects (font (size 1.27 1.27)) (justify left))
     )
@@
       (project "UpgradeBoard"
         (path "/32326095-4589-49eb-bfdc-5004b37213a0/3e08591f-9f75-4f14-b240-40be088c15b2"
-          (reference "C?") (unit 1)
+          (reference "C20") (unit 1)
         )
       )
@@
   (symbol (lib_id "Device:C_Polarized") (at 110.49 152.4 180) (unit 1)
     (in_bom yes) (on_board yes) (dnp no) (fields_autoplaced)
-    (property "Reference" "C?" (at 114.3 152.0189 0)
+    (property "Reference" "C21" (at 114.3 152.0189 0)
       (effects (font (size 1.27 1.27)) (justify right))
     )
@@
       (project "UpgradeBoard"
         (path "/32326095-4589-49eb-bfdc-5004b37213a0/3e08591f-9f75-4f14-b240-40be088c15b2"
-          (reference "C?") (unit 1)
+          (reference "C21") (unit 1)
         )
       )
@@
   (symbol (lib_id "Device:R") (at 92.71 156.21 90) (unit 1)
     (in_bom yes) (on_board yes) (dnp no) (fields_autoplaced)
-    (property "Reference" "R?" (at 92.71 149.86 90)
+    (property "Reference" "R21" (at 92.71 149.86 90)
       (effects (font (size 1.27 1.27)))
     )
@@
       (project "UpgradeBoard"
         (path "/32326095-4589-49eb-bfdc-5004b37213a0/3e08591f-9f75-4f14-b240-40be088c15b2"
-          (reference "R?") (unit 1)
+          (reference "R21") (unit 1)
         )
       )
@@
   (symbol (lib_id "Device:C_Polarized") (at 111.76 134.62 180) (unit 1)
     (in_bom yes) (on_board yes) (dnp no) (fields_autoplaced)
-    (property "Reference" "C?" (at 115.57 134.2389 0)
+    (property "Reference" "C22" (at 115.57 134.2389 0)
       (effects (font (size 1.27 1.27)) (justify right))
     )
@@
       (project "UpgradeBoard"
         (path "/32326095-4589-49eb-bfdc-5004b37213a0/3e08591f-9f75-4f14-b240-40be088c15b2"
-          (reference "C?") (unit 1)
+          (reference "C22") (unit 1)
         )
       )

Commit message: updated components
added footprint and jlcpcb component number
Parts:
- removed C19, C20: 0.1u, symbol Device:C
- removed C21, C22: 47u, symbol Device:C_Polarized
- removed R21: 100, symbol Device:R
- added C2 (x2): 0.1u, Capacitor_SMD:C_0805_2012Metric, symbol Device:C
- added C3 (x2): 47u, Capacitor_SMD:C_2220_5650Metric, symbol Device:C_Polarized
- added R57: 100, Resistor_SMD:R_0805_2012Metric, symbol Device:R
- R56: renamed from R20; footprint (none) -> Resistor_SMD:R_0805_2012Metric; Desc (none) -> 100R 1% RC12H 0805; JLC (none) -> C17408
Connections:
- net +10.8V: now also C2.2, C3.1, R57.2
- net +12V: now also R57.1
- net -10.8V: now also C2.1, C3.2
- net GND: now also C2.1, C2.2, C3.1, C3.2
