File: UpgradeBoard/AudioConnectors.kicad_sch (KiCad schematic)
At the start: 7 parts, among them J1 AudioJack3_Ground

Commit message: psucorrection
Parts:
- renumbered C14 to C?, C13 to C?, J1 to J?, R18 to R?, R22 to R?, R21 to R?, R17 to R?

Commit message: updated components
added footprint and jlcpcb component number
Parts:
- C? (x2): footprint (none) -> Capacitor_SMD:C_0603_1608Metric; Desc (none) -> 100PF 2% NP0 63V; JLC (none) -> C576781
- R? (x2): footprint (none) -> Resistor_SMD:R_0805_2012Metric; Desc (none) -> 47K 1/10W 5%; JLC (none) -> C2759457
- R? (x2): footprint (none) -> Resistor_SMD:R_0805_2012Metric; Desc (none) -> 4K7 1/10W 5%; JLC (none) -> C380775

Commit message: more components definition
Parts:
- J?: footprint (none) -> Connector_Audio:Jack_3.5mm_CUI_SJ-3524-SMT_Horizontal
Changed lines of the file:
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@@
       (effects (font (size 1.27 1.27)))
     )
-    (property "Footprint" "" (at 77.47 137.16 0)
+    (property "Footprint" "Connector_Audio:Jack_3.5mm_CUI_SJ-3524-SMT_Horizontal" (at 77.47 137.16 0)
       (effects (font (size 1.27 1.27)) hide)
     )
