File: UpgradeBoard/Demux.kicad_sch (KiCad schematic)
At the start: 18 parts, among them U2 4053, U3 4053

Commit message: friday update
new hierarchical sheets, cabling, switching for main demux
Connections:
- net A-MUTE renamed INPUTCTRL
Changed lines of the file:
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@@
     (effects (font (size 1.27 1.27)) (justify right))
   )
-  (hierarchical_label "A-MUTE" (shape input) (at 102.87 77.47 180) (fields_autoplaced)
+  (hierarchical_label "INPUTCTRL" (shape input) (at 102.87 77.47 180) (fields_autoplaced)
     (effects (font (size 1.27 1.27)) (justify right))
   )

Commit message: psucorrection
Parts:
- renumbered C15 to C1, C24 to C10, C16 to C2, C17 to C3, C18 to C4, C19 to C5, C20 to C6, C21 to C7, C22 to C8, C23 to C9, R25 to R4, R26 to R5, R27 to R6, R28 to R7, U2 to U1, U3 to U2

Commit message: updated components
added footprint and jlcpcb component number
Parts:
- removed C1: 0.1u, symbol Device:C
- removed C10, C6, C7, C8, C9: 4.7u, symbol Device:C_Polarized
- removed R5: 10k, symbol Device:R
- removed R7: 150, symbol Device:R
- added C31: 0.1u, Capacitor_SMD:C_0805_2012Metric, symbol Device:C
- added C36, C37, C38, C39, C40: 4.7u, Capacitor_SMD:C_1206_3216Metric, symbol Device:C_Polarized
- added R53: 10k, Resistor_SMD:R_0603_1608Metric, symbol Device:R
- added R55: 150, Resistor_SMD:R_0805_2012Metric, symbol Device:R
- C32: renamed from C2; footprint (none) -> Capacitor_SMD:C_0805_2012Metric; Desc (none) -> 100NF 10% X7R 0805 50V; JLC (none) -> C2929181
- C33: renamed from C3; footprint (none) -> Capacitor_SMD:C_2220_5650Metric; Desc (none) -> 47UF 20% 25V; JLC (none) -> C600189
- C34: renamed from C4; footprint (none) -> Capacitor_SMD:C_2220_5650Metric; Desc (none) -> 47UF 20% 25V; JLC (none) -> C600189
- C35: renamed from C5; footprint (none) -> Capacitor_SMD:C_1206_3216Metric; Desc (none) -> 4,7UF 50V 20%; JLC (none) -> C915818
- D1, D2: Desc (none) -> MTZJ7,5C
- R52: renamed from R4; footprint (none) -> Resistor_SMD:R_0603_1608Metric; Desc (none) -> 10K 1% 0,1W; JLC (none) -> C25804
- R54: renamed from R6; footprint (none) -> Resistor_SMD:R_0805_2012Metric; Desc (none) -> 150R 5% 0,5W; JLC (none) -> C2988914
- renumbered U1 to U4, U2 to U5
Connections:
- net -12V: now also R55.2
- net GND: now also C31.2
- net ODC: now also C39.2
- net ODR: now also R53.2
- net ODSL: now also C37.2
- net ODSR: now also C38.2
- net ODSUB: now also C40.2
- net at C32.1, C34.2, D2.2 (A)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: now also R55.1
- net at U4.4 (Z): now also C37.1
- net at U5.14 (X): now also C38.1
- net at C33.1, D1.1 (K), R54.1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: now also C31.1
- net at U5.15 (Y): now also C39.1
- net at U5.4 (Z): now also C40.1
- net at U4.15 (Y): now also C36.1
- new net: C36.2, R53.1

Commit message: more components definition
Parts:
- D1, D2: footprint (none) -> Diode_SMD:D_0603_1608Metric
- U4, U5: footprint (none) -> Package_SO:TSSOP-16_4.4x5mm_P0.65mm; JLC (none) -> C131090
Changed lines of the file:
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@@
       (effects (font (size 1.27 1.27)) (justify left))
     )
-    (property "Footprint" "" (at 198.12 139.7 0)
+    (property "Footprint" "Diode_SMD:D_0603_1608Metric" (at 198.12 139.7 0)
       (effects (font (size 1.27 1.27)) hide)
     )
@@
       (effects (font (size 1.27 1.27)) (justify left))
     )
-    (property "Footprint" "" (at 139.7 128.27 0)
-      (effects (font (size 1.27 1.27)) hide)
-    )
-    (property "Datasheet" "http://www.intersil.com/content/dam/Intersil/documents/cd40/cd4051bms-52bms-53bms.pdf" (at 139.7 128.27 0)
+    (property "Footprint" "Package_SO:TSSOP-16_4.4x5mm_P0.65mm" (at 139.7 128.27 0)
+      (effects (font (size 1.27 1.27)) hide)
+    )
+    (property "Datasheet" "https://datasheet.lcsc.com/lcsc/1809192232_Nexperia-74HCT4053PW-118_C131090.pdf" (at 139.7 128.27 0)
+      (effects (font (size 1.27 1.27)) hide)
+    )
+    (property "JLC" "C131090" (at 139.7 128.27 0)
       (effects (font (size 1.27 1.27)) hide)
     )
@@
       (effects (font (size 1.27 1.27)) (justify left))
     )
-    (property "Footprint" "" (at 139.7 64.77 0)
-      (effects (font (size 1.27 1.27)) hide)
-    )
-    (property "Datasheet" "http://www.intersil.com/content/dam/Intersil/documents/cd40/cd4051bms-52bms-53bms.pdf" (at 139.7 64.77 0)
+    (property "Footprint" "Package_SO:TSSOP-16_4.4x5mm_P0.65mm" (at 139.7 64.77 0)
+      (effects (font (size 1.27 1.27)) hide)
+    )
+    (property "Datasheet" "https://datasheet.lcsc.com/lcsc/1809192232_Nexperia-74HCT4053PW-118_C131090.pdf" (at 139.7 64.77 0)
+      (effects (font (size 1.27 1.27)) hide)
+    )
+    (property "JLC" "C131090" (at 139.7 64.77 0)
       (effects (font (size 1.27 1.27)) hide)
     )
@@
       (effects (font (size 1.27 1.27)) (justify right))
     )
-    (property "Footprint" "" (at 198.12 154.94 0)
-      (effects (font (size 1.27 1.27)) hide)
-    )
+    (property "Footprint" "Diode_SMD:D_0603_1608Metric" (at 198.12 154.94 0)
+      (effects (font (size 1.27 1.27)) hide)
+    )
