File: UpgradeBoard/OpAmp.kicad_sch (KiCad schematic)
At the start: 21 parts, among them U1 RC4558

Commit message: psucorrection
Parts:
- renumbered C1 to C11, C2 to C12, C3 to C13, C4 to C14, C5 to C15, C6 to C16, C7 to C17, C8 to C18, R3 to R10, R4 to R11, R5 to R12, R6 to R13, R7 to R14, R8 to R15, R9 to R16, R10 to R17, R11 to R18, R12 to R19, R1 to R8, R2 to R9, U1 to U3

Commit message: updated components
added footprint and jlcpcb component number
Parts:
- removed C15: 47p, symbol Device:C
- removed C17, C18: 4.7u, symbol Device:C_Polarized
- removed R13, R8, R9: 100k, symbol Device:R
- removed R15: 1k, symbol Device:R
- removed R19: 4.7k, symbol Device:R
- added C11: 47p, Capacitor_SMD:C_0805_2012Metric, symbol Device:C
- added C13, C14: 4.7u, Capacitor_SMD:C_1206_3216Metric, symbol Device:C_Polarized
- added R16, R21: 100k, Resistor_SMD:R_1206_3216Metric, symbol Device:R
- added R23: 1k, Resistor_SMD:R_0603_1608Metric, symbol Device:R
- added R25: 12k, Resistor_SMD:R_1206_3216Metric, symbol Device:R
- added R27: 4.7k, Resistor_SMD:R_0805_2012Metric, symbol Device:R
- C10: renamed from C14; footprint (none) -> Capacitor_SMD:C_0805_2012Metric; Desc (none) -> 100NF 10% X7R 0805 50V; JLC (none) -> C2929181
- C12: renamed from C16; footprint (none) -> Capacitor_SMD:C_0805_2012Metric; Desc (none) -> 47PF 1% NP0 63V; JLC (none) -> C376889
- C7: renamed from C11; footprint (none) -> Capacitor_SMD:C_1206_3216Metric; Desc (none) -> 4,7UF 50V 20%; JLC (none) -> C915818
- C8: renamed from C12; footprint (none) -> Capacitor_SMD:C_1206_3216Metric; Desc (none) -> 4,7UF 50V 20%; JLC (none) -> C915818
- C9: renamed from C13; footprint (none) -> Capacitor_SMD:C_0805_2012Metric; Desc (none) -> 100NF 10% X7R 0805 50V; JLC (none) -> C2929181
- R17: value 12k -> 100k; footprint (none) -> Resistor_SMD:R_1206_3216Metric; Desc (none) -> 100K 1% 0,1W; JLC (none) -> C965069
- R18: renamed from R10; Desc (none) -> 10K 5% 1/10W
- R19: renamed from R11; Desc (none) -> 10K 5% 1/10W
- R20: renamed from R12; footprint (none) -> Resistor_SMD:R_1206_3216Metric; Desc (none) -> 100K 1% 0,1W; JLC (none) -> C965069
- R22: renamed from R14; footprint (none) -> Resistor_SMD:R_0603_1608Metric; Desc (none) -> 1K 5% 0,1W; JLC (none) -> C21190
- R24: renamed from R16; footprint (none) -> Resistor_SMD:R_1206_3216Metric; Desc (none) -> 12K 5% 1/10W; JLC (none) -> C2771295
- R26: renamed from R18; footprint (none) -> Resistor_SMD:R_0805_2012Metric; Desc (none) -> 4K7 5% 0,1W; JLC (none) -> C380775
- renumbered U3 to U1
Connections:
- net GND: now also R17.1, C11.1, R16.1, R21.1, R23.1
- net InA: now also R17.2
- net InB: now also R16.2
- net OutA: now also R27.2
- net at R26.1: now also C13.1
- net at R19.1, U1.3 (+): now also R21.2
- net at R24.2, U1.7: now also C11.2, C13.2
- net at U1.2 (-): now also R23.2, R25.1; no longer R17.1
- net at C12.2, U1.1: now also C14.2, R25.2; no longer R17.2
- new net: C14.1, R27.1

Commit message: more components definition
Parts:
- R18, R19: footprint (none) -> Resistor_SMD:R_1206_3216Metric
- U1: footprint (none) -> Package_SO:SOIC-8_3.9x4.9mm_P1.27mm; JLC (none) -> C406864
Changed lines of the file:
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@@
       (effects (font (size 1.27 1.27)))
     )
-    (property "Footprint" "" (at 99.06 139.192 90)
+    (property "Footprint" "Resistor_SMD:R_1206_3216Metric" (at 99.06 139.192 90)
       (effects (font (size 1.27 1.27)) hide)
     )
@@
       (effects (font (size 1.27 1.27)))
     )
-    (property "Footprint" "" (at 97.79 87.122 90)
+    (property "Footprint" "Resistor_SMD:R_1206_3216Metric" (at 97.79 87.122 90)
       (effects (font (size 1.27 1.27)) hide)
     )
@@
       (effects (font (size 1.27 1.27)) (justify left))
     )
-    (property "Footprint" "" (at 115.57 58.42 0)
+    (property "Footprint" "Package_SO:SOIC-8_3.9x4.9mm_P1.27mm" (at 115.57 58.42 0)
       (effects (font (size 1.27 1.27)) hide)
     )
     (property "Datasheet" "http://www.ti.com/lit/ds/symlink/rc4558.pdf" (at 115.57 58.42 0)
+      (effects (font (size 1.27 1.27)) hide)
+    )
+    (property "JLC" "C406864" (at 115.57 58.42 0)
       (effects (font (size 1.27 1.27)) hide)
     )
@@
       (effects (font (size 1.27 1.27)))
     )
-    (property "Footprint" "" (at 125.73 91.44 0)
+    (property "Footprint" "Package_SO:SOIC-8_3.9x4.9mm_P1.27mm" (at 125.73 91.44 0)
       (effects (font (size 1.27 1.27)) hide)
     )
     (property "Datasheet" "http://www.ti.com/lit/ds/symlink/rc4558.pdf" (at 125.73 91.44 0)
+      (effects (font (size 1.27 1.27)) hide)
+    )
+    (property "JLC" "C406864" (at 125.73 91.44 0)
       (effects (font (size 1.27 1.27)) hide)
     )
@@
       (effects (font (size 1.27 1.27)))
     )
-    (property "Footprint" "" (at 127 143.51 0)
+    (property "Footprint" "Package_SO:SOIC-8_3.9x4.9mm_P1.27mm" (at 127 143.51 0)
       (effects (font (size 1.27 1.27)) hide)
     )
@@
       (effects (font (size 1.27 1.27)) hide)
     )
+    (property "JLC" "C406864" (at 127 143.51 0)
+      (effects (font (size 1.27 1.27)) hide)
+    )
